File: ISAtoTandyPlus/ISAtoTandyPlus.kicad_pcb (KiCad board)
At the start: 2 copper layers, 81 x 28.6 mm, 2 parts, among them J1 Bus_ISA_8bit, J3 TANDY PLUS HEADER

Commit message: Finished first pass at ISA to Tandy Plus.
Parts:
- added JP1: -5V, Jumper:SolderJumper-2_P1.3mm_Open_RoundedPad1.0x1.5mm, B.Cu at (165.1, 123.2)
- added JP2: AUDIO_IN, Jumper:SolderJumper-2_P1.3mm_Open_RoundedPad1.0x1.5mm, B.Cu at (157.5, 123.2)
- added JP3: ~DACK3, Jumper:SolderJumper-2_P1.3mm_Open_RoundedPad1.0x1.5mm, B.Cu at (139.7, 123.2)
- added JP4: DRQ3, Jumper:SolderJumper-2_P1.3mm_Open_RoundedPad1.0x1.5mm, B.Cu at (137.2, 123.2)
- added JP5: ~DACK1, Jumper:SolderJumper-2_P1.3mm_Open_RoundedPad1.0x1.5mm, B.Cu at (134.6, 123.2)
- added JP6: DRQ1, Jumper:SolderJumper-2_P1.3mm_Open_RoundedPad1.0x1.5mm, B.Cu at (132.1, 123.2)
- added JP7: IRQ5, Jumper:SolderJumper-2_P1.3mm_Open_RoundedPad1.0x1.5mm, B.Cu at (119.4, 123.2)
Connections:
- J3 pad 15: ~DACK3 -> Net-(J3-Pad15)
- J3 pad 16: DRQ3 -> Net-(J3-Pad16)
- J3 pad 17: ~DACK1 -> Net-(J3-Pad17)
- J3 pad 18: DRQ1 -> Net-(J3-Pad18)
- J3 pad 23: IRQ5 -> Net-(J3-Pad23)
- J3 pad 5: -5V -> Net-(J3-Pad5)
- J3 pad 8: UNUSED_THRU -> Net-(J3-Pad8)
Routing:
- net -5V: track 20.3 -> 14.0 mm
- net ~DACK3: track 20.3 -> 14.6 mm
- net ~DACK1: track 20.3 -> 14.6 mm
- net UNUSED_THRU: track 20.3 -> 14.6 mm
- net IRQ5: track 20.3 -> 14.6 mm
- net DRQ3: track 20.3 -> 14.6 mm
- net DRQ1: track 20.3 -> 14.6 mm
- net Net-(J3-Pad8): track 0.00 -> 4.45 mm
- net Net-(J3-Pad23): track 0.00 -> 4.45 mm
- net Net-(J3-Pad18): track 0.00 -> 4.45 mm
- net Net-(J3-Pad17): track 0.00 -> 4.45 mm
- net Net-(J3-Pad16): track 0.00 -> 4.45 mm
- net Net-(J3-Pad15): track 0.00 -> 4.45 mm
- net Net-(J3-Pad5): track 0.00 -> 3.81 mm
Other:
- board text added: "Allows testing of Tandy 1000 EX/HX cards in a regular ISA slot. Intended for use with an ISA riser card. Not intended for permanent installation."
- board text added: "ISA to Tandy Plus Adapter"
- board text added: "The Tandy 1000 EX/HX do not pass through all ISA bus signals. Bridge the solder jumpers to pass the signals through anyway."

Commit message: Continuing work on ISA riser card.
Other:
- board text added: "Tandy 1000 EX/HX models do not pass through all ISA bus signals. Bridge the solder jumpers to pass the signals through anyway."
- board text removed: "The Tandy 1000 EX/HX do not pass through all ISA bus signals. Bridge the solder jumpers to pass the signals through anyway."
