File: Riser/Riser.sch (KiCad schematic (older format))
At the start: 15 parts, among them J1 Bus_ISA_8bit, J2 Bus_ISA_8bit, J3 GND Hook, J4 GND Hook, J5 GND Hook

Commit message: Continuing work on ISA riser card.
Parts:
- removed F5: M205 or bridge, 00Custom:Fuseholder5x20_horiz_open_universal_Type-III, symbol Device:Fuse
- removed R5: 0.1R, 1W or bridge, Resistor_THT:R_Axial_DIN0922_L20.0mm_D9.0mm_P30.48mm_Horizontal, symbol Device:R
- added J6A1, J6B1, J7A1, J7B1: Conn_01x01, TestPoint:TestPoint_THTPad_D3.0mm_Drill1.5mm, symbol Connector_Generic:Conn_01x01
- J1, J2: symbol 00Common:Bus_ISA_8bit -> 00Common:Bus_ISA_8bit_For_Pass_Through
Connections:
- net +12V renamed 12V_IN
- net -12V renamed -12V_IN
- net -5V renamed -5V_IN
- removed net GND: J1.1 (GND), J1.10 (GND), J1.31 (GND), J2.1 (GND), J2.10 (GND), J2.31 (GND), J3.1 (Pin_1), J3.2 (Pin_2), J4.1 (Pin_1), J4.2 (Pin_2), J5.1 (Pin_1), J5.2 (Pin_2)
- net VCC renamed VCC2_IN
- net VCC2_IN: now also J6A1.1 (Pin_1); no longer J1.3 (VCC)
- net VCC_OUT_1 renamed VCC2_OUT
- net VCC2_OUT: now also J7A1.1 (Pin_1)
- net VCC_OUT_2 renamed VCC1_OUT
- net VCC1_OUT: now also J7B1.1 (Pin_1)
- new net GND1: J1.1 (GND1), J2.1 (GND1), J3.1 (Pin_1), J3.2 (Pin_2)
- new net GND2: J1.10 (GND2), J2.10 (GND2), J4.1 (Pin_1), J4.2 (Pin_2)
- new net GND3: J1.31 (GND3), J2.31 (GND3), J5.1 (Pin_1), J5.2 (Pin_2)
- new net VCC1_IN: J1.3 (VCC1), J6B1.1 (Pin_1)
Other:
- moved on the sheet: F2, F3, F4, R2, R3, R4

Commit message: Finished first pass on riser card.
Parts:
- added H1, H2: MountingHole_Pad, MountingHole:MountingHole_3.5mm_Pad, symbol Mechanical:MountingHole_Pad
- J3, J4, J5: footprint Connector_PinHeader_2.54mm:PinHeader_1x02_P2.54mm_Vertical -> 00Custom:GroundHook
Connections:
- net GND1: now also H1.1, H2.1
Changed lines of the file:
@@
 F 0 "J3" H 4880 5142 50  0000 L CNN
 F 1 "GND Hook" H 4880 5051 50  0000 L CNN
-F 2 "Connector_PinHeader_2.54mm:PinHeader_1x02_P2.54mm_Vertical" H 4800 5150 50  0001 C CNN
+F 2 "00Custom:GroundHook" H 4800 5150 50  0001 C CNN
 F 3 "~" H 4800 5150 50  0001 C CNN
 	1    4800 5150
@@
 F 0 "J4" H 4880 5692 50  0000 L CNN
 F 1 "GND Hook" H 4880 5601 50  0000 L CNN
-F 2 "Connector_PinHeader_2.54mm:PinHeader_1x02_P2.54mm_Vertical" H 4800 5700 50  0001 C CNN
+F 2 "00Custom:GroundHook" H 4800 5700 50  0001 C CNN
 F 3 "~" H 4800 5700 50  0001 C CNN
 	1    4800 5700
@@
 F 0 "J5" H 4880 6192 50  0000 L CNN
 F 1 "GND Hook" H 4880 6101 50  0000 L CNN
-F 2 "Connector_PinHeader_2.54mm:PinHeader_1x02_P2.54mm_Vertical" H 4800 6200 50  0001 C CNN
+F 2 "00Custom:GroundHook" H 4800 6200 50  0001 C CNN
 F 3 "~" H 4800 6200 50  0001 C CNN
 	1    4800 6200
@@
 	4450 5700 4350 5700
 Connection ~ 4450 5700
+$Comp
+L Mechanical:MountingHole_Pad H1
+U 1 1 608E34EA
+P 6100 5150
+F 0 "H1" V 6054 5300 50  0000 L CNN
+F 1 "MountingHole_Pad" V 6145 5300 50  0000 L CNN
+F 2 "MountingHole:MountingHole_3.5mm_Pad" H 6100 5150 50  0001 C CNN
+F 3 "~" H 6100 5150 50  0001 C CNN
+	1    6100 5150
+	0    1    1    0
+$EndComp
+$Comp
+L Mechanical:MountingHole_Pad H2
+U 1 1 608E3C9B
+P 6100 5400
+F 0 "H2" V 6054 5550 50  0000 L CNN
+F 1 "MountingHole_Pad" V 6145 5550 50  0000 L CNN
+F 2 "MountingHole:MountingHole_3.5mm_Pad" H 6100 5400 50  0001 C CNN
+F 3 "~" H 6100 5400 50  0001 C CNN
+	1    6100 5400
+	0    1    1    0
+$EndComp
+Text GLabel 5800 5150 0    50   Input ~ 0
+GND1
+Wire Wire Line
+	6000 5150 5900 5150
+Wire Wire Line
+	5900 5150 5900 5400
+Wire Wire Line
+	5900 5400 6000 5400
+Wire Wire Line
+	5900 5150 5800 5150
+Connection ~ 5900 5150
 $EndSCHEMATC
