File: Riser/Riser.kicad_pcb (KiCad board)
At the start: 2 copper layers, 99.9 x 99.9 mm, 17 parts, among them J1 Bus_ISA_8bit, J2 Bus_ISA_8bit, J3 GND Hook, J4 GND Hook, J5 GND Hook

Commit message: Continuing work on ISA riser card.
Parts:
- removed F5: M205 or bridge, 00Custom:Fuseholder5x20_horiz_open_universal_Type-III
- removed MH4: MH, MountingHole:MountingHole_3.5mm_Pad
- removed R5: 0.1R, 1W or bridge, Resistor_THT:R_Axial_DIN0922_L20.0mm_D9.0mm_P30.48mm_Horizontal
- added J6A1: Conn_01x01, TestPoint:TestPoint_THTPad_D3.0mm_Drill1.5mm, F.Cu at (104.8, 128.9)
- added J6B1: Conn_01x01, TestPoint:TestPoint_THTPad_D3.0mm_Drill1.5mm, F.Cu at (170.2, 128.9)
- added J7A1: Conn_01x01, TestPoint:TestPoint_THTPad_D3.0mm_Drill1.5mm, F.Cu at (105.4, 54.0)
- added J7B1: Conn_01x01, TestPoint:TestPoint_THTPad_D3.0mm_Drill1.5mm, F.Cu at (168.9, 54.0)
- added MH1: MountingHole_3.5mm_Pad, MountingHole:MountingHole_3.5mm_Pad, F.Cu at (192.9, 51.2)
- MH2: value MH -> MountingHole_3.5mm_Pad
- moved J4 120.1 mm to (139.1, 69.8)
- moved J3 115.0 mm to (189.2, 74.9)
- moved MH2 65.5 mm to (192.9, 116.7)
- moved J5 39.0 mm to (99.1, 73.7)
- moved F2 3.81 mm to (174.0, 102.2)
- moved F3 3.81 mm to (161.3, 102.2)
- moved F4 3.81 mm to (148.6, 102.2)
- moved R2 3.81 mm to (174.0, 61.0)
- moved R3 3.81 mm to (161.3, 61.0)
- moved R4 3.81 mm to (148.6, 61.0)
- moved F1 1.27 mm to (107.3, 102.2)
Connections:
- net +12V renamed 12V_IN
- net -12V renamed -12V_IN
- net -5V renamed -5V_IN
- net VCC_OUT_1 renamed VCC2_OUT
- F1 pad 2: VCC -> VCC2_IN
- J1 pad 1: GND -> GND1
- J1 pad 10: GND -> GND2
- J1 pad 29: VCC -> VCC2_IN
- J1 pad 3: VCC -> VCC1_IN
- J1 pad 31: GND -> GND3
- J2 pad 1: GND -> GND1
- J2 pad 10: GND -> GND2
- J2 pad 3: VCC_OUT_2 -> VCC1_OUT
- J2 pad 31: GND -> GND3
- J3 pad 1: GND -> GND1
- J3 pad 2: GND -> GND1
- J4 pad 1: GND -> GND2
- J4 pad 2: GND -> GND2
- J5 pad 1: GND -> GND3
- J5 pad 2: GND -> GND3
Routing:
- net GND: track 216.3 -> 0.00 mm
- net GND2: track 0.00 -> 102.6 mm
- net GND3: track 0.00 -> 92.6 mm
- net VCC: track 55.0 -> 0.00 mm
- net GND1: track 0.00 -> 42.8 mm
- net VCC2_IN: track 0.00 -> 31.5 mm
- net Net-(F3-Pad1): track 0.00 -> 25.2 mm
- net Net-(F2-Pad1): track 0.00 -> 25.2 mm
- net Net-(F4-Pad1): track 0.00 -> 25.2 mm
- net VCC_OUT_2: track 22.3 -> 0.00 mm
- net -12V_IN: track 16.9 -> 30.7 mm
- net -5V_IN: track 23.0 -> 35.3 mm
- net IRQ2: track 102.2 -> 113.3 mm
- net RESET: track 110.9 -> 101.6 mm
- net VCC1_IN: track 0.00 -> 8.89 mm
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- added copper zone on B.Cu, net GND1
Other:
- board text added: "+12V"
- board text added: "+5V"
- board text added: "-12V"
- board text added: "-5V"
- board text added: "A00"
- board text added: "A01"
- board text added: "A02"
- board text added: "A03"
- board text added: "A04"
- board text added: "A05"
- board text added: "A06"
- board text added: "A07"
- board text added: "A08"
- board text added: "A09"
- board text added: "A10"
- board text added: "A11"
- board text added: "A12"
- board text added: "A13"
- board text added: "A14"
- board text added: "A15"
- board text added: "A16"
- board text added: "A17"
- board text added: "A18"
- board text added: "A19"
- board text added: "AEN"
- board text added: "D0"
- board text added: "D1"
- board text added: "D2"
- board text added: "D3"
- board text added: "D4"
- board text added: "D5"
- board text added: "D6"
- board text added: "D7"
- board text added: "IOCH RDY"
- board text added: "IOCHCK"
- board text added: "WIRE LINK"

Commit message: Finished first pass on riser card.
Parts:
- removed MH1, MH2: MountingHole_3.5mm_Pad, MountingHole:MountingHole_3.5mm_Pad
- added H1: MountingHole_Pad, MountingHole:MountingHole_3.5mm_Pad, F.Cu at (192.9, 51.2)
- added H2: MountingHole_Pad, MountingHole:MountingHole_3.5mm_Pad, F.Cu at (192.9, 116.7)
- J3, J4, J5: footprint Connector_PinHeader_2.54mm:PinHeader_1x02_P2.54mm_Vertical -> 00Custom:GroundHook
- moved J3 5.43 mm to (187.3, 69.8)
- moved J5 3.81 mm to (99.1, 69.8)
Routing:
- net VCC2_OUT: track 16.4 -> 19.6 mm
- net 12V_OUT: track 16.7 -> 19.9 mm
- net -5V_OUT: track 22.2 -> 25.3 mm
- net -12V_OUT: track 15.7 -> 18.8 mm
- net VCC1_OUT: track 8.26 -> 7.62 mm
Other:
- board text added: "12V"
- board text added: "ALE"
- board text added: "All fuses M205 or wire link"
- board text added: "All resistors 0.1 ohm or wire link"
- board text added: "CLK"
- board text added: "Copyright (C) 2021 Titanium Studios Pty Ltd Creative Commons Attribution-ShareAlike 4.0 International https://github.com/JayesonLS/ISA-Cards/"
- board text added: "Current (A) = Voltage (V) across resistor * 0.1 CAUTION: Do not connect oscilloscope common ground clip to resistor. Instead clip to the ground hook and use oscilliscope differential input to measure current."
- board text added: "DRQ1"
- board text added: "DRQ2"
- board text added: "DRQ3"
- board text added: "FOR 8 BIT ISA Version 1.0"
- board text added: "GND"
- board text added: "IRQ3"
- board text added: "IRQ4"
- board text added: "IRQ5"
- board text added: "IRQ6"
- board text added: "IRQ7"
- board text added: "OSC"
- board text added: "RESET"
- board text added: "RISER"
- board text added: "Solder connector pins flush on other side first. Then bend pins before soldering this side."
- board text added: "Solder connector pins flush this side first. Then bend pins before soldering other side."
- board text added: "TC"
- board text added: "UNUSED"
- board text added: "Use bracket from generic IDE to CF adatper used for PCI slot mounting. 12.7mm (0.5") standoffs required."
- board text added: "~DACK0"
- board text added: "~DACK1"
- board text added: "~DACK2"
- board text added: "~DACK3"
- board text added: "~IOR"
- board text added: "~IOW"
- board text added: "~MEMR"
- board text added: "~MEMW"

Commit message: Updates to Riser PCB - not sure what they are?
Other:
- board text added: "Use bracket from generic IDE to CF adapter used for PCI slot mounting. 14mm of standoff spacing is required."
- board text removed: "Use bracket from generic IDE to CF adatper used for PCI slot mounting. 12.7mm (0.5") standoffs required."
