File: Template/Template.sch (KiCad schematic (older format))
At the start: 3 parts, among them J1 IDE_CONNECTOR, J2 CF Adapter Power, J3 Bus_ISA_8bit

Commit message: Fix location of CF adapter power for all boards that use it. Also the mounting holes in the schematic for the same boards. Finishing touches to Tandy 1000 Essentials.
Parts:
- added H1, H2, H3, H4: MountingHole_Pad, MountingHole:MountingHole_3.5mm_Pad, symbol Mechanical:MountingHole_Pad
- J2: footprint Connector_PinHeader_2.54mm:PinHeader_1x02_P2.54mm_Vertical -> Connector_PinSocket_2.54mm:PinSocket_1x01_P2.54mm_Vertical; symbol Connector_Generic:Conn_01x02 -> Connector_Generic:Conn_01x01
Connections:
- net GND: no longer J2.2 (Pin_2)
Changed lines of the file:
@@
 	950  4500 1500 4500
 $Comp
-L Connector_Generic:Conn_01x02 J2
+L Connector_Generic:Conn_01x01 J2
 U 1 1 603ED503
 P 7250 3750
 F 0 "J2" H 7330 3742 50  0000 L CNN
 F 1 "CF Adapter Power" H 7330 3651 50  0000 L CNN
-F 2 "Connector_PinHeader_2.54mm:PinHeader_1x02_P2.54mm_Vertical" H 7250 3750 50  0001 C CNN
+F 2 "Connector_PinSocket_2.54mm:PinSocket_1x01_P2.54mm_Vertical" H 7250 3750 50  0001 C CNN
 F 3 "~" H 7250 3750 50  0001 C CNN
 	1    7250 3750
@@
 $EndComp
 $Comp
-L power:GND #PWR0107
-U 1 1 603EF04F
-P 7050 3850
-F 0 "#PWR0107" H 7050 3600 50  0001 C CNN
-F 1 "GND" H 7055 3677 50  0000 C CNN
-F 2 "" H 7050 3850 50  0001 C CNN
-F 3 "" H 7050 3850 50  0001 C CNN
-	1    7050 3850
-	1    0    0    -1
-$EndComp
-$Comp
 L 00Common:IDE_CONNECTOR J1
 U 1 1 603E88FA
@@
 	1    0    0    -1
 $EndComp
+$Comp
+L Mechanical:MountingHole_Pad H1
+U 1 1 608FC9D0
+P 7200 4100
+F 0 "H1" V 7154 4250 50  0000 L CNN
+F 1 "MountingHole_Pad" V 7245 4250 50  0000 L CNN
+F 2 "MountingHole:MountingHole_3.5mm_Pad" H 7200 4100 50  0001 C CNN
+F 3 "~" H 7200 4100 50  0001 C CNN
+	1    7200 4100
+	0    1    1    0
+$EndComp
+$Comp
+L Mechanical:MountingHole_Pad H2
+U 1 1 608FD692
+P 7200 4350
+F 0 "H2" V 7154 4500 50  0000 L CNN
+F 1 "MountingHole_Pad" V 7245 4500 50  0000 L CNN
+F 2 "MountingHole:MountingHole_3.5mm_Pad" H 7200 4350 50  0001 C CNN
+F 3 "~" H 7200 4350 50  0001 C CNN
+	1    7200 4350
+	0    1    1    0
+$EndComp
+$Comp
+L Mechanical:MountingHole_Pad H3
+U 1 1 608FD8F9
+P 7200 4600
+F 0 "H3" V 7154 4750 50  0000 L CNN
+F 1 "MountingHole_Pad" V 7245 4750 50  0000 L CNN
+F 2 "MountingHole:MountingHole_3.5mm_Pad" H 7200 4600 50  0001 C CNN
+F 3 "~" H 7200 4600 50  0001 C CNN
+	1    7200 4600
+	0    1    1    0
+$EndComp
+$Comp
+L Mechanical:MountingHole_Pad H4
+U 1 1 608FDAF1
+P 7200 4850
+F 0 "H4" V 7154 5000 50  0000 L CNN
+F 1 "MountingHole_Pad" V 7245 5000 50  0000 L CNN
+F 2 "MountingHole:MountingHole_3.5mm_Pad" H 7200 4850 50  0001 C CNN
+F 3 "~" H 7200 4850 50  0001 C CNN
+	1    7200 4850
+	0    1    1    0
+$EndComp
 $EndSCHEMATC
