File: Template/Template.kicad_pcb (KiCad board)
At the start: 2 copper layers, 99.9 x 99.9 mm, 7 parts, among them J1 IDE_CONNECTOR, J2 CF Adapter Power, J3 Bus_ISA_8bit

Commit message: Fix location of CF adapter power for all boards that use it. Also the mounting holes in the schematic for the same boards. Finishing touches to Tandy 1000 Essentials.
Parts:
- H1: renamed from MH1; value MH -> MountingHole_Pad
- H2: renamed from MH2; value MH -> MountingHole_Pad
- H3: renamed from MH3; value MH -> MountingHole_Pad
- H4: renamed from MH4; value MH -> MountingHole_Pad
- J2: footprint Connector_PinHeader_2.54mm:PinHeader_1x02_P2.54mm_Vertical -> Connector_PinSocket_2.54mm:PinSocket_1x01_P2.54mm_Vertical
- moved J2 7.62 mm to (182.0, 59.8)

Commit message: Template: Fix orientation of CF adapter header (rotate 180 degrees).
Parts:
- moved J1 48.3 mm to (165.1, 108.1), turned to 180 degrees
