File: TandyPlusTemplate/TandyPlusTemplate.sch (KiCad schematic (older format))
At the start: 3 parts, among them J1 Input BUS, J2 Passthrough Bus Short, J3 Passthrough Bus Tall

Commit message: Work on Tandy Plus template.
Parts:
- J1: footprint Connector_PinSocket_2.54mm:PinSocket_2x31_P2.54mm_Vertical -> 00Custom:TandyPlusSocket
- J2: footprint Connector_PinHeader_2.54mm:PinHeader_2x31_P2.54mm_Vertical -> 00Custom:TandyPlusShortPins
- J3: footprint Connector_PinHeader_2.54mm:PinHeader_2x31_P2.54mm_Vertical -> 00Custom:TandyPlusLongPins
Changed lines of the file:
@@
 F 0 "J1" H 2000 4317 50  0000 C CNN
 F 1 "Input BUS" H 2000 4226 50  0000 C CNN
-F 2 "Connector_PinSocket_2.54mm:PinSocket_2x31_P2.54mm_Vertical" H 2000 2550 50  0001 C CNN
+F 2 "00Custom:TandyPlusSocket" H 2000 2550 50  0001 C CNN
 F 3 "https://en.wikipedia.org/wiki/Industry_Standard_Architecture" H 2000 2550 50  0001 C CNN
 	1    2000 2550
@@
 F 0 "J2" H 4700 4317 50  0000 C CNN
 F 1 "Passthrough Bus Short" H 4700 4226 50  0000 C CNN
-F 2 "Connector_PinHeader_2.54mm:PinHeader_2x31_P2.54mm_Vertical" H 4700 2550 50  0001 C CNN
+F 2 "00Custom:TandyPlusShortPins" H 4700 2550 50  0001 C CNN
 F 3 "https://en.wikipedia.org/wiki/Industry_Standard_Architecture" H 4700 2550 50  0001 C CNN
 	1    4700 2550
@@
 F 0 "J3" H 7400 4317 50  0000 C CNN
 F 1 "Passthrough Bus Tall" H 7400 4226 50  0000 C CNN
-F 2 "Connector_PinHeader_2.54mm:PinHeader_2x31_P2.54mm_Vertical" H 7400 2550 50  0001 C CNN
+F 2 "00Custom:TandyPlusLongPins" H 7400 2550 50  0001 C CNN
 F 3 "https://en.wikipedia.org/wiki/Industry_Standard_Architecture" H 7400 2550 50  0001 C CNN
 	1    7400 2550

Commit message: Complete first pass at Tandy Plus template by adding bracket details.
Parts:
- added H1, H2, H3, H4, H5, H6: MountingHole_Pad, MountingHole:MountingHole_3.5mm_Pad, symbol Mechanical:MountingHole_Pad
Changed lines of the file:
@@
 Text GLabel 1000 2450 0    39   Input ~ 0
 ~DACK3
+$Comp
+L Mechanical:MountingHole_Pad H1
+U 1 1 60D532A5
+P 9600 2000
+F 0 "H1" V 9554 2150 50  0000 L CNN
+F 1 "MountingHole_Pad" V 9645 2150 50  0000 L CNN
+F 2 "MountingHole:MountingHole_3.5mm_Pad" H 9600 2000 50  0001 C CNN
+F 3 "~" H 9600 2000 50  0001 C CNN
+	1    9600 2000
+	0    1    1    0
+$EndComp
+$Comp
+L Mechanical:MountingHole_Pad H2
+U 1 1 60D54339
+P 9600 2200
+F 0 "H2" V 9554 2350 50  0000 L CNN
+F 1 "MountingHole_Pad" V 9645 2350 50  0000 L CNN
+F 2 "MountingHole:MountingHole_3.5mm_Pad" H 9600 2200 50  0001 C CNN
+F 3 "~" H 9600 2200 50  0001 C CNN
+	1    9600 2200
+	0    1    1    0
+$EndComp
+$Comp
+L Mechanical:MountingHole_Pad H3
+U 1 1 60D635F3
+P 9600 2400
+F 0 "H3" V 9554 2550 50  0000 L CNN
+F 1 "MountingHole_Pad" V 9645 2550 50  0000 L CNN
+F 2 "MountingHole:MountingHole_3.5mm_Pad" H 9600 2400 50  0001 C CNN
+F 3 "~" H 9600 2400 50  0001 C CNN
+	1    9600 2400
+	0    1    1    0
+$EndComp
+$Comp
+L Mechanical:MountingHole_Pad H4
+U 1 1 60D63887
+P 9600 2600
+F 0 "H4" V 9554 2750 50  0000 L CNN
+F 1 "MountingHole_Pad" V 9645 2750 50  0000 L CNN
+F 2 "MountingHole:MountingHole_3.5mm_Pad" H 9600 2600 50  0001 C CNN
+F 3 "~" H 9600 2600 50  0001 C CNN
+	1    9600 2600
+	0    1    1    0
+$EndComp
+$Comp
+L Mechanical:MountingHole_Pad H5
+U 1 1 60D7304E
+P 9600 2800
+F 0 "H5" V 9554 2950 50  0000 L CNN
+F 1 "MountingHole_Pad" V 9645 2950 50  0000 L CNN
+F 2 "MountingHole:MountingHole_3.5mm_Pad" H 9600 2800 50  0001 C CNN
+F 3 "~" H 9600 2800 50  0001 C CNN
+	1    9600 2800
+	0    1    1    0
+$EndComp
+$Comp
+L Mechanical:MountingHole_Pad H6
+U 1 1 60D732FE
+P 9600 3000
+F 0 "H6" V 9554 3150 50  0000 L CNN
+F 1 "MountingHole_Pad" V 9645 3150 50  0000 L CNN
+F 2 "MountingHole:MountingHole_3.5mm_Pad" H 9600 3000 50  0001 C CNN
+F 3 "~" H 9600 3000 50  0001 C CNN
+	1    9600 3000
+	0    1    1    0
+$EndComp
 $EndSCHEMATC
