File: EX-HX-Combo/EX-HX-Combo.sch (KiCad schematic (older format))
At the start: 36 parts, among them CN1 DB9 Male, J1 IDE_CONNECTOR, J2 CF Adapter Power, J3 Bus_Tandy_Plus, J4 Addresses, J5 Addresses, J6 Addresses, J7 Addresses, U1 BIOS FLASH, U2 74HCT245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

Commit message: EX-HX-Combo: Add a pass at the IO decode logic.
Connections:
- net labels added: ~BASE_RAM_ENABLE, ~CS3~_ATA, ~UART_ENABLE
- net labels removed: BASE_RAM_ENABLE, COM_ENABLE
- wire segments 200 -> 198
Changed lines of the file:
@@
 Text GLabel 14450 1900 2    50   Input ~ 0
 D7_BUF
-Text GLabel 8200 3600 2    39   Input ~ 0
+Text GLabel 8200 3700 2    39   Input ~ 0
 ~IOR~_DELAYED
 Text GLabel 2650 3450 2    50   Input ~ 0
@@
 	1    0    0    -1
 $EndComp
-Text GLabel 8200 3700 2    39   Input ~ 0
+Text GLabel 8200 3800 2    39   Input ~ 0
 ~BUFF_READ
 Text GLabel 7200 3500 0    39   Input ~ 0
@@
 Wire Wire Line
 	11250 5100 11250 5300
-Text GLabel 8200 3500 2    39   Input ~ 0
+Text GLabel 8200 3600 2    39   Input ~ 0
 ~MEMR~_DELAYED
 $Comp
@@
 Wire Wire Line
 	4550 4450 4550 4550
-Text GLabel 4650 4350 0    50   Input ~ 0
-COM_ENABLE
-Text GLabel 7200 3300 0    50   Input ~ 0
-COM_ENABLE
-Text GLabel 8200 4000 2    39   Input ~ 0
-~IOR
+Text GLabel 4650 4350 0    39   Input ~ 0
+~UART_ENABLE
+Text GLabel 7200 3300 0    39   Input ~ 0
+~UART_ENABLE
 Text GLabel 8200 1650 2    39   Input ~ 0
 ~RESET
@@
 Text GLabel 8200 3300 2    39   Input ~ 0
 ~CS1~_ATA
-Text GLabel 8200 3400 2    39   Input ~ 0
+Text GLabel 8200 3500 2    39   Input ~ 0
 ~UART_CS
 Text GLabel 8200 1350 2    39   Input ~ 0
@@
 Text GLabel 5150 1400 2    50   Input ~ 0
 ATA_ADDR_JUMPER
-Text GLabel 8200 3800 2    50   Input ~ 0
+Text GLabel 8200 3900 2    50   Input ~ 0
 MEMR_DECODE
 Text GLabel 8200 1250 2    39   Input ~ 0
@@
 Text Notes 5350 4650 0    50   ~ 0
 RTC Enable
-Text GLabel 7200 1250 0    50   Input ~ 0
-BASE_RAM_ENABLE
-Text GLabel 4650 2350 0    50   Input ~ 0
-BASE_RAM_ENABLE
+Text GLabel 7200 1250 0    39   Input ~ 0
+~BASE_RAM_ENABLE
+Text GLabel 4650 2350 0    39   Input ~ 0
+~BASE_RAM_ENABLE
 Text GLabel 7200 1350 0    50   Input ~ 0
 BASE_RAM_SIZE
@@
 Wire Wire Line
 	1550 3350 1050 3350
-Text GLabel 8200 3900 2    50   Input ~ 0
+Text GLabel 8200 4000 2    50   Input ~ 0
 AEN
 Text GLabel 13150 6500 0    50   Input ~ 0
@@
 Text GLabel 13150 6400 0    50   Input ~ 0
 A17_MAPPED
-$Comp
-L power:VCC #PWR0177
-U 1 1 60D680E6
-P 11250 6050
-F 0 "#PWR0177" H 11250 5900 50  0001 C CNN
-F 1 "VCC" H 11265 6223 50  0000 C CNN
-F 2 "" H 11250 6050 50  0001 C CNN
-F 3 "" H 11250 6050 50  0001 C CNN
-	1    11250 6050
-	1    0    0    -1
-$EndComp
-Wire Wire Line
-	10700 6150 11250 6150
-Wire Wire Line
-	11250 6150 11250 6050
 Text GLabel 4650 1400 0    50   Input ~ 0
 ROM_ADDR_JUMPER
@@
 Wire Notes Line
 	12250 3950 12250 7050
+Text GLabel 8200 3400 2    39   Input ~ 0
+~CS3~_ATA
+Text GLabel 10700 6150 2    39   Input ~ 0
+~CS3~_ATA
 $EndSCHEMATC

Commit message: EX-HX-Combo: Add a pass at the memory decode logic.
Connections:
- net labels added: UMB_DECODE, UMB_SIZE, ~UMB_ENABLE
- net labels removed: ROM_ADDR_JUMPER, UMB_SIZE_0, UMB_SIZE_1
- wire segments 198 -> 200
- no-connect marks 41 -> 43
Changed lines of the file:
@@
 Text GLabel 7200 3300 0    39   Input ~ 0
 ~UART_ENABLE
-Text GLabel 8200 1650 2    39   Input ~ 0
+Text GLabel 8200 1850 2    39   Input ~ 0
 ~RESET
-Text GLabel 8200 1750 2    50   Input ~ 0
+Text GLabel 8200 1950 2    50   Input ~ 0
 RESET
 Text GLabel 8200 3300 2    39   Input ~ 0
@@
 Text GLabel 8200 1250 2    39   Input ~ 0
 ~CE~_BIOS_DECODE
-Text GLabel 8200 1850 2    50   Input ~ 0
+Text GLabel 8200 1650 2    50   Input ~ 0
 MEMR_DECODE
 $Comp
@@
 Wire Wire Line
 	5250 3250 5250 3150
-Text GLabel 5150 3350 2    50   Input ~ 0
-UMB_SIZE_1
-Text GLabel 4650 3350 0    50   Input ~ 0
-UMB_SIZE_0
 Text GLabel 8200 1450 2    50   Input ~ 0
 A18_MAPPED
@@
 Text GLabel 7200 1350 0    50   Input ~ 0
 BASE_RAM_SIZE
-Text GLabel 7200 1450 0    50   Input ~ 0
-UMB_SIZE_0
+Text GLabel 7200 1450 0    39   Input ~ 0
+~UMB_ENABLE
 Text GLabel 7200 1550 0    50   Input ~ 0
-UMB_SIZE_1
+UMB_SIZE
 $Comp
 L power:+12V #PWR0175
@@
 Text GLabel 13150 6400 0    50   Input ~ 0
 A17_MAPPED
-Text GLabel 4650 1400 0    50   Input ~ 0
-ROM_ADDR_JUMPER
-Text GLabel 8200 1950 2    50   Input ~ 0
-ROM_ADDR_JUMPER
 $Comp
 L Device:CP C10
@@
 $EndComp
 $Comp
-L power:VCC #PWR?
+L power:VCC #PWR0121
 U 1 1 60E3DBDE
 P 13400 7550
-F 0 "#PWR?" H 13400 7400 50  0001 C CNN
+F 0 "#PWR0121" H 13400 7400 50  0001 C CNN
 F 1 "VCC" H 13415 7723 50  0000 C CNN
 F 2 "" H 13400 7550 50  0001 C CNN
@@
 $EndComp
 $Comp
-L power:GND #PWR?
+L power:GND #PWR0122
 U 1 1 60E3E530
 P 13400 7850
-F 0 "#PWR?" H 13400 7600 50  0001 C CNN
+F 0 "#PWR0122" H 13400 7600 50  0001 C CNN
 F 1 "GND" H 13405 7677 50  0000 C CNN
 F 2 "" H 13400 7850 50  0001 C CNN
@@
 Text GLabel 10700 6150 2    39   Input ~ 0
 ~CS3~_ATA
+Text Label 8550 1800 0    50   ~ 0
+UMB_DECODE
+Wire Wire Line
+	8200 1750 8550 1750
+NoConn ~ 8550 1800
+Wire Wire Line
+	8550 1750 8550 1800
+NoConn ~ 4650 1400
+Text GLabel 4650 3350 0    39   Input ~ 0
+~UMB_ENABLE
+Text GLabel 5150 3350 2    50   Input ~ 0
+UMB_SIZE
 $EndSCHEMATC

Commit message: EX-HX-Combo: Add mutple com port choices, update programmable logic to match.
Connections:
- net labels added: IOR_DECODE, UART_PORT_0, UART_PORT_1
- net labels removed: MEMR_DECODE, UMB_DECODE, ~UART_ENABLE
- wire segments 200 -> 198
- no-connect marks 43 -> 41
Changed lines of the file:
@@
 Text GLabel 14450 1900 2    50   Input ~ 0
 D7_BUF
-Text GLabel 8200 3700 2    39   Input ~ 0
+Text GLabel 8200 1750 2    39   Input ~ 0
 ~IOR~_DELAYED
 Text GLabel 2650 3450 2    50   Input ~ 0
@@
 Text GLabel 10100 2600 0    39   Input ~ 0
 ~BUFF_READ
-Text GLabel 7200 3400 0    50   Input ~ 0
+Text GLabel 8200 4000 2    50   Input ~ 0
 ATA_ADDR_JUMPER
 Text GLabel 2650 2650 2    50   Input ~ 0
@@
 	1    0    0    -1
 $EndComp
-Text GLabel 8200 3800 2    39   Input ~ 0
+Text GLabel 8200 1850 2    39   Input ~ 0
 ~BUFF_READ
 Text GLabel 7200 3500 0    39   Input ~ 0
@@
 Wire Wire Line
 	11250 5100 11250 5300
-Text GLabel 8200 3600 2    39   Input ~ 0
+Text GLabel 8200 1650 2    39   Input ~ 0
 ~MEMR~_DELAYED
 $Comp
@@
 Wire Wire Line
 	4550 4450 4550 4550
-Text GLabel 4650 4350 0    39   Input ~ 0
-~UART_ENABLE
-Text GLabel 7200 3300 0    39   Input ~ 0
-~UART_ENABLE
-Text GLabel 8200 1850 2    39   Input ~ 0
-~RESET
-Text GLabel 8200 1950 2    50   Input ~ 0
-RESET
+Text GLabel 7200 3400 0    50   Input ~ 0
+UART_PORT_1
 Text GLabel 8200 3300 2    39   Input ~ 0
 ~CS1~_ATA
@@
 Text GLabel 5150 2350 2    50   Input ~ 0
 BASE_RAM_SIZE
-Text GLabel 5150 1400 2    50   Input ~ 0
+Text GLabel 4650 4350 0    50   Input ~ 0
 ATA_ADDR_JUMPER
-Text GLabel 8200 3900 2    50   Input ~ 0
-MEMR_DECODE
+Text GLabel 8200 3600 2    50   Input ~ 0
+IOR_DECODE
 Text GLabel 8200 1250 2    39   Input ~ 0
 ~CE~_BIOS_DECODE
-Text GLabel 8200 1650 2    50   Input ~ 0
-MEMR_DECODE
 $Comp
 L Connector_Generic:Conn_02x03_Odd_Even J6
@@
 Wire Wire Line
 	1550 3350 1050 3350
-Text GLabel 8200 4000 2    50   Input ~ 0
+Text GLabel 8200 3900 2    50   Input ~ 0
 AEN
 Text GLabel 13150 6500 0    50   Input ~ 0
@@
 Text GLabel 10700 6150 2    39   Input ~ 0
 ~CS3~_ATA
-Text Label 8550 1800 0    50   ~ 0
-UMB_DECODE
-Wire Wire Line
-	8200 1750 8550 1750
-NoConn ~ 8550 1800
-Wire Wire Line
-	8550 1750 8550 1800
-NoConn ~ 4650 1400
 Text GLabel 4650 3350 0    39   Input ~ 0
 ~UMB_ENABLE
 Text GLabel 5150 3350 2    50   Input ~ 0
 UMB_SIZE
+Text GLabel 7200 3300 0    50   Input ~ 0
+UART_PORT_0
+Text GLabel 8200 3800 2    50   Input ~ 0
+RESET
+Text GLabel 8200 3700 2    39   Input ~ 0
+~RESET
+Text GLabel 8200 1950 2    50   Input ~ 0
+IOR_DECODE
+Text GLabel 4650 1400 0    50   Input ~ 0
+UART_PORT_0
+Text GLabel 5150 1400 2    50   Input ~ 0
+UART_PORT_1
 $EndSCHEMATC

Commit message: Add COM IRQ selection to EX-HX-Combo.
Parts:
- added J8: UART IRQ, Connector_PinHeader_2.54mm:PinHeader_2x03_P2.54mm_Vertical, symbol Connector_Generic:Conn_02x03_Odd_Even
- J4: value Addresses -> UART port
- J5: value Addresses -> Base RAM
- J6: value Addresses -> UMB
- J7: value Addresses -> ATA & RTC
Connections:
- net labels added: IRQ2, IRQ3, UART_IRQ
- wire segments 198 -> 206
- no-connect marks 41 -> 39

Commit message: EX=HX-Combo: Mods preparing for board layout. Made some changes for SMT production, including changes to how the jumpers are implemented. Updated GAL logic to match,
Parts:
- removed H1, H2, H3, H4: MountingHole_Pad, MountingHole:MountingHole_3.5mm_Pad, symbol Mechanical:MountingHole_Pad
- removed J2: CF Adapter Power, Connector_PinSocket_2.54mm:PinSocket_1x02_P2.54mm_Vertical, symbol Connector_Generic:Conn_01x02
- removed J4: UART port, Connector_PinHeader_2.54mm:PinHeader_2x03_P2.54mm_Vertical, symbol Connector_Generic:Conn_02x03_Odd_Even
- removed J5: Base RAM, Connector_PinHeader_2.54mm:PinHeader_2x03_P2.54mm_Vertical, symbol Connector_Generic:Conn_02x03_Odd_Even
- removed J6: UMB, Connector_PinHeader_2.54mm:PinHeader_2x03_P2.54mm_Vertical, symbol Connector_Generic:Conn_02x03_Odd_Even
- removed J7: ATA & RTC, Connector_PinHeader_2.54mm:PinHeader_2x03_P2.54mm_Vertical, symbol Connector_Generic:Conn_02x03_Odd_Even
- removed J8: UART IRQ, Connector_PinHeader_2.54mm:PinHeader_2x03_P2.54mm_Vertical, symbol Connector_Generic:Conn_02x03_Odd_Even
- added J2: Jumpers, symbol Connector_Generic:Conn_02x09_Odd_Even
- added R1, R2, R3, R4, R5, R6, R7: 10K, Resistor_SMD:R_1206_3216Metric, symbol Device:R
- BAT1: footprint Battery:BatteryHolder_Keystone_103_1x20mm -> Battery:BatteryHolder_Keystone_1060_1x2032
- C1, C2, C3, C4, C5: footprint Capacitor_THT:C_Disc_D6.0mm_W2.5mm_P5.00mm -> Capacitor_SMD:C_1206_3216Metric
- C6, C7, C8, C9: footprint Capacitor_THT:C_Disc_D5.1mm_W3.2mm_P5.00mm -> Capacitor_SMD:C_1206_3216Metric
- J1: footprint Connector_PinSocket_2.54mm:PinSocket_2x20_P2.54mm_Vertical -> Connector_PinSocket_2.00mm:PinSocket_2x22_P2.00mm_Horizontal; symbol 00Common:IDE_CONNECTOR -> 00Common:IDE_CONNECTOR_44
- J3: footprint 00Custom:BUS_XT -> 00Custom:TandyPlusSocket
- U6: footprint Package_DIP:DIP-40_W15.24mm_Socket -> Package_QFP:LQFP-48_7x7mm_P0.5mm; symbol Interface_UART:16550 -> 00Common:16550_48
- U8, U9: footprint (none) -> Package_DIP:DIP-20_W7.62mm_Socket
Connections:
- net labels added: BASE_RAM_ENABLE, UART_S0, UART_S1, UMB_ENABLE
- net labels removed: IRQ2, UART_PORT_0, UART_PORT_1, ~BASE_RAM_ENABLE, ~CE~_BIOS, ~UMB_ENABLE
- wire segments 206 -> 208
- no-connect marks 39 -> 41
Other:
- note removed: "RTC Enable"

Commit message: Mods to EX-HX-Combo.
Parts:
- removed C10: 22uF, Capacitor_THT:CP_Radial_D7.5mm_P2.50mm, symbol Device:CP
- removed U3: 1.8432 MHz, 00Custom:Crystal_DIP8_DIP14, symbol 00Common:CRYSTAL_OSCILLATOR_BOTH_SIZES
- added U3: 1.8432 MHz, Oscillator:Oscillator_SMD_SeikoEpson_SG8002CA-4Pin_7.0x5.0mm, symbol Oscillator:SG-7050CAN
- C10: renamed from C11; value 22uF -> 100uF; footprint Capacitor_THT:CP_Radial_D7.5mm_P2.50mm -> Capacitor_Tantalum_SMD:CP_EIA-3528-15_AVX-H
- C11: renamed from C12; value 4.7uF -> 10uF; footprint Capacitor_THT:CP_Radial_D7.5mm_P2.50mm -> Capacitor_Tantalum_SMD:CP_EIA-3216-18_Kemet-A
- C12: renamed from C13; value 4.7uF -> 10uF; footprint Capacitor_THT:CP_Radial_D7.5mm_P2.50mm -> Capacitor_Tantalum_SMD:CP_EIA-3216-18_Kemet-A
- J2: footprint (none) -> Connector_PinHeader_2.54mm:PinHeader_2x09_P2.54mm_Vertical_SMD
- U2, U7: footprint Package_DIP:DIP-20_W7.62mm_Socket -> Package_SO:SOIC-20W_7.5x12.8mm_P1.27mm
Connections:
- net GND: now also U3.2 (GND)
- net UART_XIN: now also U3.3 (OUT)
- net VCC: now also U3.1 (~ST), U3.4 (VCC)
Changed lines of the file:
@@
 F 0 "U2" H 10800 2950 50  0000 C CNN
 F 1 "74HCT245" H 10800 2850 50  0000 C CNN
-F 2 "Package_DIP:DIP-20_W7.62mm_Socket" H 10600 2200 50  0001 C CNN
+F 2 "Package_SO:SOIC-20W_7.5x12.8mm_P1.27mm" H 10600 2200 50  0001 C CNN
 F 3 "http://www.ti.com/lit/gpn/sn74LS245" H 10600 2200 50  0001 C CNN
 	1    10600 2200
@@
 F 0 "U7" H 6300 9000 50  0000 C CNN
 F 1 "GD75232N" H 6400 8900 50  0000 C CNN
-F 2 "Package_DIP:DIP-20_W7.62mm_Socket" H 6050 7500 50  0001 C CIN
+F 2 "Package_SO:SOIC-20W_7.5x12.8mm_P1.27mm" H 6050 7500 50  0001 C CIN
 F 3 "http://www.ti.com/lit/ds/symlink/gd75232.pdf" H 5550 8300 50  0001 C CNN
 	1    6050 8300
@@
 F 3 "" H 12400 7550 50  0001 C CNN
 	1    12400 7550
-	1    0    0    -1
-$EndComp
-$Comp
-L power:VCC #PWR0148
-U 1 1 60D203AE
-P 12900 7550
-F 0 "#PWR0148" H 12900 7400 50  0001 C CNN
-F 1 "VCC" H 12915 7723 50  0000 C CNN
-F 2 "" H 12900 7550 50  0001 C CNN
-F 3 "" H 12900 7550 50  0001 C CNN
-	1    12900 7550
-	1    0    0    -1
-$EndComp
-$Comp
-L power:GND #PWR0149
-U 1 1 60D203B8
-P 12900 7850
-F 0 "#PWR0149" H 12900 7600 50  0001 C CNN
-F 1 "GND" H 12905 7677 50  0000 C CNN
-F 2 "" H 12900 7850 50  0001 C CNN
-F 3 "" H 12900 7850 50  0001 C CNN
-	1    12900 7850
 	1    0    0    -1
 $EndComp
@@
 Wire Wire Line
 	2350 8900 2350 7450
-$Comp
-L 00Common:CRYSTAL_OSCILLATOR_BOTH_SIZES U3
-U 1 1 60D203D6
-P 7450 6050
-F 0 "U3" H 7450 6537 60  0000 C CNN
-F 1 "1.8432 MHz" H 7450 6431 60  0000 C CNN
-F 2 "00Custom:Crystal_DIP8_DIP14" H 6950 6050 60  0001 C CNN
-F 3 "" H 6950 6050 60  0000 C CNN
-	1    7450 6050
-	1    0    0    -1
-$EndComp
-$Comp
-L power:GND #PWR0151
-U 1 1 60D203E0
-P 6700 6350
-F 0 "#PWR0151" H 6700 6100 50  0001 C CNN
-F 1 "GND" H 6705 6177 50  0000 C CNN
-F 2 "" H 6700 6350 50  0001 C CNN
-F 3 "" H 6700 6350 50  0001 C CNN
-	1    6700 6350
-	1    0    0    -1
-$EndComp
-$Comp
-L power:VCC #PWR0152
-U 1 1 60D203EB
-P 6700 5750
-F 0 "#PWR0152" H 6700 5600 50  0001 C CNN
-F 1 "VCC" H 6715 5923 50  0000 C CNN
-F 2 "" H 6700 5750 50  0001 C CNN
-F 3 "" H 6700 5750 50  0001 C CNN
-	1    6700 5750
-	1    0    0    -1
-$EndComp
-$Comp
-L power:VCC #PWR0153
-U 1 1 60D203F5
-P 8200 5750
-F 0 "#PWR0153" H 8200 5600 50  0001 C CNN
-F 1 "VCC" H 8215 5923 50  0000 C CNN
-F 2 "" H 8200 5750 50  0001 C CNN
-F 3 "" H 8200 5750 50  0001 C CNN
-	1    8200 5750
-	1    0    0    -1
-$EndComp
-Wire Wire Line
-	8200 5750 8200 5850
-Wire Wire Line
-	8200 5850 8100 5850
-Wire Wire Line
-	6700 5750 6700 5850
-Wire Wire Line
-	6700 5850 6800 5850
-Wire Wire Line
-	8100 6050 8200 6050
-Wire Wire Line
-	8200 6050 8200 5850
-Connection ~ 8200 5850
-Wire Wire Line
-	6800 6050 6700 6050
-Wire Wire Line
-	6800 6250 6700 6250
-Wire Wire Line
-	6700 6250 6700 6350
-Text GLabel 8100 6250 2    50   Input ~ 0
-UART_XIN
 Text GLabel 2650 9300 0    50   Input ~ 0
 UART_XIN
@@
 	1    0    0    -1
 $EndComp
-$Comp
-L power:GND #PWR0157
-U 1 1 60D204FA
-P 13950 7850
-F 0 "#PWR0157" H 13950 7600 50  0001 C CNN
-F 1 "GND" H 13955 7677 50  0000 C CNN
-F 2 "" H 13950 7850 50  0001 C CNN
-F 3 "" H 13950 7850 50  0001 C CNN
-	1    13950 7850
-	1    0    0    -1
-$EndComp
-$Comp
-L power:GND #PWR0158
-U 1 1 60D20504
-P 14900 7550
-F 0 "#PWR0158" H 14900 7300 50  0001 C CNN
-F 1 "GND" H 14905 7377 50  0000 C CNN
-F 2 "" H 14900 7550 50  0001 C CNN
-F 3 "" H 14900 7550 50  0001 C CNN
-	1    14900 7550
-	1    0    0    -1
-$EndComp
-$Comp
-L power:+12V #PWR0159
-U 1 1 60D2050E
-P 13950 7550
-F 0 "#PWR0159" H 13950 7400 50  0001 C CNN
-F 1 "+12V" H 13965 7723 50  0000 C CNN
-F 2 "" H 13950 7550 50  0001 C CNN
-F 3 "" H 13950 7550 50  0001 C CNN
-	1    13950 7550
-	1    0    0    -1
-$EndComp
-$Comp
-L power:-12V #PWR0160
-U 1 1 60D20518
-P 14450 7850
-F 0 "#PWR0160" H 14450 7950 50  0001 C CNN
-F 1 "-12V" H 14465 8023 50  0000 C CNN
-F 2 "" H 14450 7850 50  0001 C CNN
-F 3 "" H 14450 7850 50  0001 C CNN
-	1    14450 7850
-	-1   0    0    1
-$EndComp
-$Comp
-L Device:CP C13
-U 1 1 60D20522
-P 14450 7700
-F 0 "C13" H 14568 7746 50  0000 L CNN
-F 1 "4.7uF" H 14568 7655 50  0000 L CNN
-F 2 "Capacitor_THT:CP_Radial_D7.5mm_P2.50mm" H 14488 7550 50  0001 C CNN
-F 3 "~" H 14450 7700 50  0001 C CNN
-	1    14450 7700
-	1    0    0    -1
-$EndComp
-Wire Wire Line
-	14450 7550 14450 7450
-Wire Wire Line
-	14450 7450 14900 7450
-Wire Wire Line
-	14900 7450 14900 7550
 Text Label 6700 8600 0    50   ~ 0
 SER_PIN1
@@
 Text Label 6700 7900 0    50   ~ 0
 SER_PIN9
-Wire Wire Line
-	6700 6050 6700 5850
-Connection ~ 6700 5850
 Wire Wire Line
 	13250 2700 12650 2700
@@
 A17_MAPPED
 $Comp
-L Device:CP C10
-U 1 1 60D20354
-P 12900 7700
-F 0 "C10" H 13018 7746 50  0000 L CNN
-F 1 "22uF" H 13018 7655 50  0000 L CNN
-F 2 "Capacitor_THT:CP_Radial_D7.5mm_P2.50mm" H 12938 7550 50  0001 C CNN
-F 3 "~" H 12900 7700 50  0001 C CNN
-	1    12900 7700
-	1    0    0    -1
-$EndComp
-$Comp
-L Device:CP C12
-U 1 1 60D204F0
-P 13950 7700
-F 0 "C12" H 14068 7746 50  0000 L CNN
-F 1 "4.7uF" H 14068 7655 50  0000 L CNN
-F 2 "Capacitor_THT:CP_Radial_D7.5mm_P2.50mm" H 13988 7550 50  0001 C CNN
-F 3 "~" H 13950 7700 50  0001 C CNN
-	1    13950 7700
-	1    0    0    -1
-$EndComp
-$Comp
 L power:VCC #PWR0121
 U 1 1 60E3DBDE
@@
 	1    0    0    -1
 $EndComp
-$Comp
-L Device:CP C11
-U 1 1 60E3E53A
-P 13400 7700
-F 0 "C11" H 13518 7746 50  0000 L CNN
-F 1 "22uF" H 13518 7655 50  0000 L CNN
-F 2 "Capacitor_THT:CP_Radial_D7.5mm_P2.50mm" H 13438 7550 50  0001 C CNN
-F 3 "~" H 13400 7700 50  0001 C CNN
-	1    13400 7700
-	1    0    0    -1
-$EndComp
-Wire Notes Line
-	8200 7150 15050 7150
-Wire Notes Line
-	15050 7150 15050 8150
-Wire Notes Line
-	15050 8150 8200 8150
 Wire Notes Line
 	8200 8250 8200 11100
@@
 F 0 "J2" H 10650 10500 50  0000 C CNN
 F 1 "Jumpers" H 10650 10400 50  0000 C CNN
-F 2 "" H 10600 9900 50  0001 C CNN
+F 2 "Connector_PinHeader_2.54mm:PinHeader_2x09_P2.54mm_Vertical_SMD" H 10600 9900 50  0001 C CNN
 F 3 "~" H 10600 9900 50  0001 C CNN
 	1    10600 9900
@@
 Connection ~ 9100 10100
 NoConn ~ 1550 1350
+Wire Wire Line
+	14900 7450 14900 7550
+Wire Wire Line
+	14450 7450 14900 7450
+Wire Wire Line
+	14450 7550 14450 7450
+$Comp
+L power:-12V #PWR0160
+U 1 1 60D20518
+P 14450 7850
+F 0 "#PWR0160" H 14450 7950 50  0001 C CNN
+F 1 "-12V" H 14465 8023 50  0000 C CNN
+F 2 "" H 14450 7850 50  0001 C CNN
+F 3 "" H 14450 7850 50  0001 C CNN
+	1    14450 7850
+	-1   0    0    1
+$EndComp
+$Comp
+L power:+12V #PWR0159
+U 1 1 60D2050E
+P 13950 7550
+F 0 "#PWR0159" H 13950 7400 50  0001 C CNN
+F 1 "+12V" H 13965 7723 50  0000 C CNN
+F 2 "" H 13950 7550 50  0001 C CNN
+F 3 "" H 13950 7550 50  0001 C CNN
+	1    13950 7550
+	1    0    0    -1
+$EndComp
+$Comp
+L power:GND #PWR0158
+U 1 1 60D20504
+P 14900 7550
+F 0 "#PWR0158" H 14900 7300 50  0001 C CNN
+F 1 "GND" H 14905 7377 50  0000 C CNN
+F 2 "" H 14900 7550 50  0001 C CNN
+F 3 "" H 14900 7550 50  0001 C CNN
+	1    14900 7550
+	1    0    0    -1
+$EndComp
+$Comp
+L power:GND #PWR0157
+U 1 1 60D204FA
+P 13950 7850
+F 0 "#PWR0157" H 13950 7600 50  0001 C CNN
+F 1 "GND" H 13955 7677 50  0000 C CNN
+F 2 "" H 13950 7850 50  0001 C CNN
+F 3 "" H 13950 7850 50  0001 C CNN
+	1    13950 7850
+	1    0    0    -1
+$EndComp
+Wire Notes Line
+	15050 8150 8200 8150
+Wire Notes Line
+	15050 7150 15050 8150
+Wire Notes Line
+	8200 7150 15050 7150
+$Comp
+L power:GND #PWR0151
+U 1 1 60D203E0
+P 7550 6400
+F 0 "#PWR0151" H 7550 6150 50  0001 C CNN
+F 1 "GND" H 7555 6227 50  0000 C CNN
+F 2 "" H 7550 6400 50  0001 C CNN
+F 3 "" H 7550 6400 50  0001 C CNN
+	1    7550 6400
+	1    0    0    -1
+$EndComp
+$Comp
+L power:VCC #PWR0152
+U 1 1 60D203EB
+P 7150 5800
+F 0 "#PWR0152" H 7150 5650 50  0001 C CNN
+F 1 "VCC" H 7165 5973 50  0000 C CNN
+F 2 "" H 7150 5800 50  0001 C CNN
+F 3 "" H 7150 5800 50  0001 C CNN
+	1    7150 5800
+	1    0    0    -1
+$EndComp
+$Comp
+L power:VCC #PWR0153
+U 1 1 60D203F5
+P 7550 5800
+F 0 "#PWR0153" H 7550 5650 50  0001 C CNN
+F 1 "VCC" H 7565 5973 50  0000 C CNN
+F 2 "" H 7550 5800 50  0001 C CNN
+F 3 "" H 7550 5800 50  0001 C CNN
+	1    7550 5800
+	1    0    0    -1
+$EndComp
+Wire Wire Line
+	7250 6100 7150 6100
+$Comp
+L Oscillator:SG-7050CAN U3
+U 1 1 6125B3CC
+P 7550 6100
+F 0 "U3" H 7650 6450 50  0000 L CNN
+F 1 "1.8432 MHz" H 7650 6350 50  0000 L CNN
+F 2 "Oscillator:Oscillator_SMD_SeikoEpson_SG8002CA-4Pin_7.0x5.0mm" H 8250 5750 50  0001 C CNN
+F 3 "https://support.epson.biz/td/api/doc_check.php?dl=brief_SG7050CAN&lang=en" H 7450 6100 50  0001 C CNN
+	1    7550 6100
+	1    0    0    -1
+$EndComp
+Wire Wire Line
+	7150 5800 7150 6100
+Text GLabel 7850 6100 2    50   Input ~ 0
+UART_XIN
+$Comp
+L Device:CP C10
+U 1 1 60E3E53A
+P 13400 7700
+F 0 "C10" H 13518 7746 50  0000 L CNN
+F 1 "100uF" H 13518 7655 50  0000 L CNN
+F 2 "Capacitor_Tantalum_SMD:CP_EIA-3528-15_AVX-H" H 13438 7550 50  0001 C CNN
+F 3 "~" H 13400 7700 50  0001 C CNN
+	1    13400 7700
+	1    0    0    -1
+$EndComp
+$Comp
+L Device:CP C11
+U 1 1 60D204F0
+P 13950 7700
+F 0 "C11" H 14068 7746 50  0000 L CNN
+F 1 "10uF" H 14068 7655 50  0000 L CNN
+F 2 "Capacitor_Tantalum_SMD:CP_EIA-3216-18_Kemet-A" H 13988 7550 50  0001 C CNN
+F 3 "~" H 13950 7700 50  0001 C CNN
+	1    13950 7700
+	1    0    0    -1
+$EndComp
+$Comp
+L Device:CP C12
+U 1 1 60D20522
+P 14450 7700
+F 0 "C12" H 14568 7746 50  0000 L CNN
+F 1 "10uF" H 14568 7655 50  0000 L CNN
+F 2 "Capacitor_Tantalum_SMD:CP_EIA-3216-18_Kemet-A" H 14488 7550 50  0001 C CNN
+F 3 "~" H 14450 7700 50  0001 C CNN
+	1    14450 7700
+	1    0    0    -1
+$EndComp
 $EndSCHEMATC
