File: EX-HX-Combo/Backplate/EX-HX-Combo-Backplate.sch (KiCad schematic (older format))
At the start: 0 parts

Commit message: Work on EX-HX-Combo backplate. Made a panel, however JLCPCB can't determine the board outline and do not know how to specify the v-score across the top and bottom.
Parts:
- added H1: Serial Port Holes, 00Custom:DB9_Face_NPTH, symbol Mechanical:MountingHole
Changed lines of the file:
@@
 Comment4 ""
 $EndDescr
+$Comp
+L Mechanical:MountingHole H1
+U 1 1 611CEF27
+P 5000 5000
+F 0 "H1" H 5100 5046 50  0000 L CNN
+F 1 "Serial Port Holes" H 5100 4955 50  0000 L CNN
+F 2 "00Custom:DB9_Face_NPTH" H 5000 5000 50  0001 C CNN
+F 3 "~" H 5000 5000 50  0001 C CNN
+	1    5000 5000
+	1    0    0    -1
+$EndComp
 $EndSCHEMATC
