File: CF-Combo-Super-Lite/CF-Combo-Super-Lite.kicad_pcb (KiCad board)
At the start: 2 copper layers, 99.9 x 99.9 mm, 22 parts, among them J1 IDE_CONNECTOR, J2 CF Adapter Power, J3 Bus_ISA_8bit, J4 Addresses, J5 Addresses, U1 BIOS FLASH, U2 74HCT245, U3 GAL22V10, U4 DS1315, U5 AS6C4008-55PCN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

Commit message: Add gerbers for CF-Combo-Super-Lite.
Other:
- board text added: "KEYSTONE 103 OR SIMILAR"

Commit message: CF-Combo-Super-Lite: Add additional bypass cap to CF power. Add back in V20+ jumper (selects different flash ROM range). Add version number. Initial work setting up for JLCPCB production, however they won't assemble boards with edge connectors.
Parts:
- added C6: 0.1uF, Capacitor_THT:C_Disc_D6.0mm_W2.5mm_P5.00mm, F.Cu at (185.4, 59.8)
- U3: value GAL22V10 -> ATF/GAL22V10x-15
- renumbered C6 to C7
Connections:
- J5 pad 3: Net-(J5-Pad3) -> V20_JUMPER
- U1 pad 2: GND -> V20_JUMPER
Routing:
- net V20_JUMPER: track 0.00 -> 26.2 mm
- net ATA_ADDR_JUMPER: track 57.7 -> 63.2 mm
- net VCC: track 454.5 -> 458.0 mm
- net GND: track 344.5 -> 347.2 mm
Other:
- board text added: "8086/8088"
- board text added: "CPU TYPE"
- board text added: "JLCJLCJLCJLC"
- board text added: "V20, 286,..."
- board text added: "v1.1"
- board text removed: "UNUSED"
