File: IsaTemplate/IsaTemplate.kicad_pcb (KiCad board)
At the start: 2 copper layers, 99.9 x 99.9 mm, 7 parts, among them J1 IDE_CONNECTOR, J2 CF Adapter Power, J3 Bus_ISA_8bit

Commit message: Add Keystone 9202 holes to template.
Other:
- board text added: "Keystone 9202 hole"
Changed lines of the file:
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@@
   (general
     (thickness 1.6)
-    (drawings 26)
+    (drawings 30)
     (tracks 0)
     (zones 0)
@@
       (effects (font (size 1 1) (thickness 0.15)))
     )
+    (fp_line (start -1.27 -1.27) (end 0.635 -1.27) (layer F.Fab) (width 0.1))
+    (fp_line (start 0.635 -1.27) (end 1.27 -0.635) (layer F.Fab) (width 0.1))
+    (fp_line (start 1.27 -0.635) (end 1.27 1.27) (layer F.Fab) (width 0.1))
+    (fp_line (start 1.27 1.27) (end -1.27 1.27) (layer F.Fab) (width 0.1))
+    (fp_line (start -1.27 1.27) (end -1.27 -1.27) (layer F.Fab) (width 0.1))
+    (fp_line (start -1.33 1.33) (end 1.33 1.33) (layer F.SilkS) (width 0.12))
+    (fp_line (start -1.33 1.21) (end -1.33 1.33) (layer F.SilkS) (width 0.12))
+    (fp_line (start 1.33 1.21) (end 1.33 1.33) (layer F.SilkS) (width 0.12))
+    (fp_line (start 1.33 -1.33) (end 1.33 0) (layer F.SilkS) (width 0.12))
+    (fp_line (start 0 -1.33) (end 1.33 -1.33) (layer F.SilkS) (width 0.12))
+    (fp_line (start -1.8 -1.8) (end 1.75 -1.8) (layer F.CrtYd) (width 0.05))
+    (fp_line (start 1.75 -1.8) (end 1.75 1.75) (layer F.CrtYd) (width 0.05))
+    (fp_line (start 1.75 1.75) (end -1.8 1.75) (layer F.CrtYd) (width 0.05))
     (fp_line (start -1.8 1.75) (end -1.8 -1.8) (layer F.CrtYd) (width 0.05))
-    (fp_line (start 1.75 1.75) (end -1.8 1.75) (layer F.CrtYd) (width 0.05))
-    (fp_line (start 1.75 -1.8) (end 1.75 1.75) (layer F.CrtYd) (width 0.05))
-    (fp_line (start -1.8 -1.8) (end 1.75 -1.8) (layer F.CrtYd) (width 0.05))
-    (fp_line (start 0 -1.33) (end 1.33 -1.33) (layer F.SilkS) (width 0.12))
-    (fp_line (start 1.33 -1.33) (end 1.33 0) (layer F.SilkS) (width 0.12))
-    (fp_line (start 1.33 1.21) (end 1.33 1.33) (layer F.SilkS) (width 0.12))
-    (fp_line (start -1.33 1.21) (end -1.33 1.33) (layer F.SilkS) (width 0.12))
-    (fp_line (start -1.33 1.33) (end 1.33 1.33) (layer F.SilkS) (width 0.12))
-    (fp_line (start -1.27 1.27) (end -1.27 -1.27) (layer F.Fab) (width 0.1))
-    (fp_line (start 1.27 1.27) (end -1.27 1.27) (layer F.Fab) (width 0.1))
-    (fp_line (start 1.27 -0.635) (end 1.27 1.27) (layer F.Fab) (width 0.1))
-    (fp_line (start 0.635 -1.27) (end 1.27 -0.635) (layer F.Fab) (width 0.1))
-    (fp_line (start -1.27 -1.27) (end 0.635 -1.27) (layer F.Fab) (width 0.1))
     (fp_text user %R (at 0 1.27) (layer F.Fab)
       (effects (font (size 1 1) (thickness 0.15)))
@@
       (effects (font (size 1 1) (thickness 0.15)))
     )
+    (fp_line (start -3.81 -1.27) (end 0.27 -1.27) (layer F.Fab) (width 0.1))
+    (fp_line (start 0.27 -1.27) (end 1.27 -0.27) (layer F.Fab) (width 0.1))
+    (fp_line (start 1.27 -0.27) (end 1.27 49.53) (layer F.Fab) (width 0.1))
+    (fp_line (start 1.27 49.53) (end -3.81 49.53) (layer F.Fab) (width 0.1))
+    (fp_line (start -3.81 49.53) (end -3.81 -1.27) (layer F.Fab) (width 0.1))
+    (fp_line (start -3.87 -1.33) (end -1.27 -1.33) (layer F.SilkS) (width 0.12))
+    (fp_line (start -3.87 -1.33) (end -3.87 49.59) (layer F.SilkS) (width 0.12))
+    (fp_line (start -3.87 49.59) (end 1.33 49.59) (layer F.SilkS) (width 0.12))
+    (fp_line (start 1.33 1.27) (end 1.33 49.59) (layer F.SilkS) (width 0.12))
+    (fp_line (start -1.27 1.27) (end 1.33 1.27) (layer F.SilkS) (width 0.12))
+    (fp_line (start -1.27 -1.33) (end -1.27 1.27) (layer F.SilkS) (width 0.12))
+    (fp_line (start 1.33 -1.33) (end 1.33 0) (layer F.SilkS) (width 0.12))
+    (fp_line (start 0 -1.33) (end 1.33 -1.33) (layer F.SilkS) (width 0.12))
+    (fp_line (start -4.34 -1.8) (end 1.76 -1.8) (layer F.CrtYd) (width 0.05))
+    (fp_line (start 1.76 -1.8) (end 1.76 50) (layer F.CrtYd) (width 0.05))
+    (fp_line (start 1.76 50) (end -4.34 50) (layer F.CrtYd) (width 0.05))
     (fp_line (start -4.34 50) (end -4.34 -1.8) (layer F.CrtYd) (width 0.05))
-    (fp_line (start 1.76 50) (end -4.34 50) (layer F.CrtYd) (width 0.05))
-    (fp_line (start 1.76 -1.8) (end 1.76 50) (layer F.CrtYd) (width 0.05))
-    (fp_line (start -4.34 -1.8) (end 1.76 -1.8) (layer F.CrtYd) (width 0.05))
-    (fp_line (start 0 -1.33) (end 1.33 -1.33) (layer F.SilkS) (width 0.12))
-    (fp_line (start 1.33 -1.33) (end 1.33 0) (layer F.SilkS) (width 0.12))
-    (fp_line (start -1.27 -1.33) (end -1.27 1.27) (layer F.SilkS) (width 0.12))
-    (fp_line (start -1.27 1.27) (end 1.33 1.27) (layer F.SilkS) (width 0.12))
-    (fp_line (start 1.33 1.27) (end 1.33 49.59) (layer F.SilkS) (width 0.12))
-    (fp_line (start -3.87 49.59) (end 1.33 49.59) (layer F.SilkS) (width 0.12))
-    (fp_line (start -3.87 -1.33) (end -3.87 49.59) (layer F.SilkS) (width 0.12))
-    (fp_line (start -3.87 -1.33) (end -1.27 -1.33) (layer F.SilkS) (width 0.12))
-    (fp_line (start -3.81 49.53) (end -3.81 -1.27) (layer F.Fab) (width 0.1))
-    (fp_line (start 1.27 49.53) (end -3.81 49.53) (layer F.Fab) (width 0.1))
-    (fp_line (start 1.27 -0.27) (end 1.27 49.53) (layer F.Fab) (width 0.1))
-    (fp_line (start 0.27 -1.27) (end 1.27 -0.27) (layer F.Fab) (width 0.1))
-    (fp_line (start -3.81 -1.27) (end 0.27 -1.27) (layer F.Fab) (width 0.1))
     (fp_text user %R (at -1.27 24.13 90) (layer F.Fab)
       (effects (font (size 1 1) (thickness 0.15)))
@@
       (net 33 GND))
   )
+  (gr_text "Keystone 9202 hole" (at 190.5 130.175) (layer Cmts.User)
+    (effects (font (size 1 1) (thickness 0.15)) (justify right))
+  )
+  (gr_text "Keystone 9202 hole" (at 190.5 73.66) (layer Cmts.User)
+    (effects (font (size 1 1) (thickness 0.15)) (justify right))
+  )
+  (gr_circle (center 192.405 130.19) (end 193.905 130.19) (layer Dwgs.User) (width 0.15))
+  (gr_circle (center 192.383 73.67) (end 193.883 73.67) (layer Dwgs.User) (width 0.15))
   (gr_line (start 201.273 134.62) (end 201.273 41.22) (layer Dwgs.User) (width 0.05))
   (gr_line (start 207.01 41.22) (end 207.01 41.91) (layer Dwgs.User) (width 0.05))
