File: Tandy1000Essentials/Tandy1000Essentials.sch (KiCad schematic (older format))
At the start: 23 parts, among them J1 IDE_CONNECTOR, J2 CF Adapter Power, J3 Bus_ISA_8bit, J4 Addresses, J5 Addresses, U1 BIOS FLASH, U2 74HCT245, U3 ATF/GAL22V10x-15, U4 DS1315, U5 AS6C4008-55PCN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

Commit message: Tandy 1000 Essentials: Remove references to non-Tandy 1000 configurations.
Other:
- note added: "512K SRAM"
- note removed: "TANDY 1000 SRAM\n(OPTIONAL)"
Changed lines of the file:
@@
 Text GLabel 10200 5300 2    39   Input ~ 0
 ~MEMW
-Text Notes 8500 3750 0    79   ~ 0
-TANDY 1000 SRAM\n(OPTIONAL)
+Text Notes 8500 3600 0    79   ~ 0
+512K SRAM
 Wire Notes Line
 	8450 3450 11150 3450
