File: Tandy1000Essentials/Tandy1000Essentials.kicad_pcb (KiCad board)
At the start: 2 copper layers, 99.9 x 99.9 mm, 23 parts, among them J1 IDE_CONNECTOR, J2 CF Adapter Power, J3 Bus_ISA_8bit, J4 Addresses, J5 Addresses, U1 BIOS FLASH, U2 74HCT245, U3 ATF/GAL22V10x-15, U4 DS1315, U5 AS6C4008-55PCN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

Commit message: Update boards.
Other:
- board text added: "Created by Jayeson Lee-Steere https://github.com/ JayesonLS/ISA-Cards"
- board text removed: "Copyright (C) 2021 Titanium Studios Pty Ltd Creative Commons Attribution-ShareAlike 4.0 International https://github.com/ JayesonLS/ISA-Cards"
