File: CFSuperLite/CFSuperLite.kicad_pcb (KiCad board)
At the start: 2 copper layers, 99.9 x 99.9 mm, 23 parts, among them J1 IDE_CONNECTOR, J2 CF Adapter Power, J3 Bus_ISA_8bit, SW1 Options, U1 BIOS FLASH, U2 74HCT245, U3 ATF/GAL16V8x-15, U4 DS1315, Y1 32.768 KHz

Commit message: CFSuperLite: Add diagram describing how the tall header with long pins should be fitted to the board.
Parts:
- added REF**: PinHeader_2x20_P2.54mm_Vertical, Connector_PinHeader_2.54mm:PinHeader_2x20_P2.54mm_Vertical, F.Cu at (208.3, 73.7)
- J1: value IDE_CONNECTOR -> IDE to CF adapter
Other:
- board text added: "Assembling J1"
- board text added: "Cut/trim all pins"
- board text added: "Mount connector flush to PCB"
