File: BasicSerial/BasicSerial.kicad_pcb (KiCad board)
At the start: 2 copper layers, 99.9 x 73 mm, 15 parts, among them CN1 DB9 Male, J1 COM_SELECT, J2 IRQ_SELECT, J3 Bus_ISA_8bit, U1 16550/16C550, U2 74LS688, 74HCT688 or GAL16V8, U3 GD75232N, U4 1.8432 MHz

Commit message: Update boards.
Other:
- board text added: "Version 1.0 Created by Jayeson Lee-Steere https://github.com/ JayesonLS/ISA-Cards/"
- board text removed: "Version 1.0 Copyright (C) 2021 Titanium Studios Pty Ltd Creative Commons Attribution-ShareAlike 4.0 International https://github.com/ JayesonLS/ISA-Cards/"
