File: PCSuperCombo/PCSuperCombo.kicad_pcb (KiCad board)
At the start: 2 copper layers, 123.3 x 95 mm, 42 parts, among them CN1 DB9 Male, J1 IDE_CONNECTOR, J2 CF Adapter Power, J3 Bus_ISA_8bit, J4 LED, SW1 Options, U1 BIOS FLASH, U10 1.8432 MHz, U2 74HCT245, U3 ATF/GAL16V8x-15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

Commit message: PCSuperCombo WIP.
Parts:
- added R10: 0R, Resistor_SMD:R_1206_3216Metric, F.Cu at (120.7, 27.9)
- added R11: 0R, Resistor_SMD:R_1206_3216Metric, F.Cu at (120.7, 31.2)
- renumbered R10 to R12, R11 to R13
Connections:
- R8 pad 2: COM1_ENABLE -> V20_JUMPER
- R9 pad 2: V20_JUMPER -> COM1_ENABLE
- SW1 pad 11: ~CE~_BIOS -> GND
- SW1 pad 12: ~IOR_OR_MEMR -> ~CE~_BIOS
- SW1 pad 13: ~CARD_SEL -> ~CE~_BIOS_THRU
- SW1 pad 14: ~CE~_BIOS_THRU -> COM1_ENABLE
- SW1 pad 16: V20_JUMPER -> ~CARD_SEL
- SW1 pad 17: COM1_ENABLE -> V20_JUMPER
- SW1 pad 21: (no net) -> UMB_SIZE_0
- SW1 pad 22: (no net) -> BASE_RAM_2
- SW1 pad 23: (no net) -> BASE_RAM_1
- SW1 pad 24: (no net) -> BASE_RAM_0
- SW1 pad 9: GND -> ~IOR_OR_MEMR
- U1 pad 13: D0_BUF -> Net-(U1-Pad13)
- U1 pad 14: D1_BUF -> Net-(U1-Pad14)
- U1 pad 15: D2_BUF -> Net-(U1-Pad15)
- U1 pad 17: D3_BUF -> Net-(U1-Pad17)
- U1 pad 18: D4_BUF -> Net-(U1-Pad18)
- U1 pad 19: D5_BUF -> Net-(U1-Pad19)
- U1 pad 20: D6_BUF -> Net-(U1-Pad20)
- U1 pad 21: D7_BUF -> Net-(U1-Pad21)
- U8 pad 2: D5 -> D5_BUF
- U8 pad 3: D6 -> D6_BUF
- U8 pad 4: D7 -> D7_BUF
- U8 pad 43: D0 -> D0_BUF
- U8 pad 44: D1 -> D1_BUF
- U8 pad 45: D2 -> D2_BUF
- U8 pad 46: D3 -> D3_BUF
- U8 pad 47: D4 -> D4_BUF

Commit message: Update boards.
Other:
- board text added: "Created by Jayeson Lee-Steere https://github.com/ JayesonLS/ISA-Cards"
- board text removed: "Copyright (C) 2021 Titanium Studios Pty Ltd Creative Commons Attribution-ShareAlike 4.0 International https://github.com/ JayesonLS/ISA-Cards"
